Commit message: test to fix jazzy branch for ur examples

File: manymove_bringup/srdf/ur_with_robotiq.srdf.xacro (robot description, xacro)
@@ -3,6 +3,45 @@
   <xacro:arg name="name" default="ur"/>
   <xacro:arg name="prefix" default=""/>
-  <xacro:include filename="$(find ur_moveit_config)/srdf/ur_macro.srdf.xacro"/>
-  <xacro:ur_srdf name="$(arg name)" prefix="$(arg prefix)"/>
+  <!-- Manipulator group -->
+  <group name="ur_manipulator">
+    <chain base_link="$(arg prefix)base_link" tip_link="$(arg prefix)tool0"/>
+  </group>
+  <!-- Common joint states -->
+  <group_state name="home" group="ur_manipulator">
+    <joint name="$(arg prefix)shoulder_pan_joint" value="0"/>
+    <joint name="$(arg prefix)shoulder_lift_joint" value="-1.5707"/>
+    <joint name="$(arg prefix)elbow_joint" value="0"/>
+    <joint name="$(arg prefix)wrist_1_joint" value="0"/>
+    <joint name="$(arg prefix)wrist_2_joint" value="0"/>
+    <joint name="$(arg prefix)wrist_3_joint" value="0"/>
+  </group_state>
+  <group_state name="up" group="ur_manipulator">
+    <joint name="$(arg prefix)shoulder_pan_joint" value="0"/>
+    <joint name="$(arg prefix)shoulder_lift_joint" value="-1.5707"/>
+    <joint name="$(arg prefix)elbow_joint" value="0"/>
+    <joint name="$(arg prefix)wrist_1_joint" value="-1.5707"/>
+    <joint name="$(arg prefix)wrist_2_joint" value="0"/>
+    <joint name="$(arg prefix)wrist_3_joint" value="0"/>
+  </group_state>
+  <group_state name="test_configuration" group="ur_manipulator">
+    <joint name="$(arg prefix)shoulder_pan_joint" value="1.54"/>
+    <joint name="$(arg prefix)shoulder_lift_joint" value="-1.62"/>
+    <joint name="$(arg prefix)elbow_joint" value="1.4"/>
+    <joint name="$(arg prefix)wrist_1_joint" value="-1.2"/>
+    <joint name="$(arg prefix)wrist_2_joint" value="-1.6"/>
+    <joint name="$(arg prefix)wrist_3_joint" value="-0.11"/>
+  </group_state>
+  <!-- Disable standard UR self-collisions -->
+  <disable_collisions link1="$(arg prefix)base_link" link2="$(arg prefix)base_link_inertia" reason="Adjacent"/>
+  <disable_collisions link1="$(arg prefix)base_link_inertia" link2="$(arg prefix)shoulder_link" reason="Adjacent"/>
+  <disable_collisions link1="$(arg prefix)tool0" link2="$(arg prefix)wrist_1_link" reason="Never"/>
+  <disable_collisions link1="$(arg prefix)tool0" link2="$(arg prefix)wrist_2_link" reason="Never"/>
+  <disable_collisions link1="$(arg prefix)tool0" link2="$(arg prefix)wrist_3_link" reason="Adjacent"/>
+  <disable_collisions link1="$(arg prefix)forearm_link" link2="$(arg prefix)upper_arm_link" reason="Adjacent"/>
+  <disable_collisions link1="$(arg prefix)forearm_link" link2="$(arg prefix)wrist_1_link" reason="Adjacent"/>
+  <disable_collisions link1="$(arg prefix)shoulder_link" link2="$(arg prefix)upper_arm_link" reason="Adjacent"/>
+  <disable_collisions link1="$(arg prefix)wrist_1_link" link2="$(arg prefix)wrist_2_link" reason="Adjacent"/>
+  <disable_collisions link1="$(arg prefix)wrist_1_link" link2="$(arg prefix)wrist_3_link" reason="Never"/>
+  <disable_collisions link1="$(arg prefix)wrist_2_link" link2="$(arg prefix)wrist_3_link" reason="Adjacent"/>
   <!-- Disable collisions for rigidly attached Robotiq base -->
   <disable_collisions link1="$(arg prefix)wrist_3_link" link2="$(arg prefix)robotiq_85_base_link" reason="Adjacent"/>
